Commit message: harvester tool

File: stretch_description/urdf/stretch.urdf (robot description, URDF)
Before this commit: robot stretch_description, 42 links, 41 joints
Links:
- added link harvester_frame
- added link harvester_link, mass 0.102736408077; collision mesh filename=package://stretch_description/meshes/harvester_link.STL; visual mesh filename=package://stretch_description/meshes/harvester_link.STL
- added link pollinator_frame
Joints:
- added joint h_joint: type fixed, parent harvester_link, child harvester_frame, origin xyz=.13 -0.045 0.045 rpy=0.0 0.0 0.0
- added joint harvest: type fixed, parent link_wrist_yaw, child harvester_link, origin xyz=0.0 0 0 rpy=0 0.0 0, axis 0.0 0.0 0.0
- added joint p_joint: type fixed, parent tool_link, child pollinator_frame, origin xyz=.13 -0.045 0.045 rpy=0.0 0.0 0.0
- joint tool: origin xyz=0.0 0.0 -0.038 rpy=3.14159 0.0 -1.5708 -> xyz=0.0 0 0 rpy=0 0.0 0
